Commit message: simulate_v3.0   3d转2d后调用move_base

File: src/urdf_learn_gazebo/urdf/racecar.xacro (robot description, xacro)
@@ -2,4 +2,13 @@
 <robot name="racebot" xmlns:xacro="http://www.ros.org/wiki/xacro">
     <xacro:include filename="$(find urdf_learn_gazebo)/urdf/macros.xacro" />
+    <xacro:include filename="$(find urdf_learn_gazebo)/velodyne_description/urdf/VLP-16.urdf.xacro" />
+    <joint name="lidar_joint" type="fixed">
+      <origin xyz="0.093603 0 0.12377" />
+      <axis xyz="0 0 1" />
+      <parent link="base_link"/>
+      <child link="velodyne_base_link"/>
+    </joint>
+    <xacro:VLP-16/>
+    <robot_base_gazebo/>
     <link name="base_footprint">
     </link>
@@ -284,5 +293,5 @@
             <child link="realsense_depth"/>
     </joint>
-    <link name="lidar">
+    <!-- <link name="lidar">
         <visual>
             <geometry>
@@ -311,6 +320,6 @@
         <origin xyz="0.093603 0 0.12377" />
         <axis xyz="0 0 1" />
-    </joint>
-    <link name="imu">
+    </joint> -->
+    <!-- <link name="imu">
         <visual>
             <geometry>
@@ -339,5 +348,5 @@
         <origin xyz="0 0 0.02" />
         <axis xyz="0 0 1" />
-    </joint>
+    </joint> -->
   <xacro:include filename="$(find urdf_learn_gazebo)/urdf/racecar.gazebo" />
 </robot>
